Commit message: Replaced stretch_gazebo with stretch_control

File: stretch_control/urdf/stretch/stretch_base.xacro (robot description, xacro)
@@ -7,5 +7,5 @@
                 xyz="-0.109461304328163 -0.000741018909047708 0.0914915269429946"
                 rpy="0 0 0"/>
-            <mass value="1.0723782659782"/>
+            <mass value="${1.0723782659782}"/>
             <inertia
                 ixx="0.00310580907710135"
@@ -37,7 +37,3 @@
         </collision>
     </link>
-    <gazebo reference="base_link">
-        <mu1 value="0.0"/>
-        <mu2 value="0.0"/>
-    </gazebo>
 </robot>

File: stretch_control/urdf/stretch/stretch_head.xacro (robot description, xacro)
@@ -141,5 +141,5 @@
         </collision>
     </link>
-    <!-- Head Pan Joint -->
+    <!-- Head Tilt Joint -->
     <joint name="joint_head_tilt" type="revolute">
         <origin
@@ -151,5 +151,5 @@
         <limit effort="100" lower="-1.53" upper="0.79" velocity="1.0"/>
     </joint>
-    <!-- Head Pan Transmission block for gazebo -->
+    <!-- Head Tilt Transmission block for gazebo -->
     <transmission name="trans_head_tilt" type="SimpleTransmission">
         <type>transmission_interface/SimpleTransmission</type>

File: stretch_control/urdf/stretch/stretch_left_wheel.xacro (robot description, xacro)
@@ -7,5 +7,5 @@
                 xyz="1.2555462092223E-07 -3.54748938502514E-07 -0.0239581106165035"
                 rpy="0 0 0" />
-            <mass value="0.00356714564938459" />
+            <mass value="${0.00356714564938459}" />
             <inertia ixx="0" ixy="0" ixz="0"
                      iyy="0" iyz="0"
@@ -40,16 +40,5 @@
         <axis xyz="0 0 1" />
     </joint>
-    <!-- Left Wheel Physical Properties for Gazebo -->
-    <gazebo reference="joint_right_wheel">
-        <mu1 value="200.0"/>
-        <mu2 value="100.0"/>
-        <kp value="10000000.0"/>
-        <kd value="1.0"/>
-        <material name="">
-            <color
-                rgba="0.792156862745098 0.819607843137255 0.933333333333333 1" />
-        </material>
-    </gazebo>
-    <!-- Gazebo transmission block for simulation -->
+    <!-- Transmission block for ROS control -->
     <transmission name="trans_left_wheel">
         <type>transmission_interface/SimpleTransmission</type>

File: stretch_control/urdf/stretch/stretch_mast.xacro (robot description, xacro)
@@ -7,5 +7,5 @@
                 xyz="0.00755818572975822 0.773971284176834 0.00647313086620024"
                 rpy="0 0 0"/>
-            <mass value="0.749143203376401"/>
+            <mass value="${0.749143203376401*mast_mass}"/>
             <inertia
                 ixx="0.0709854511954588"
@@ -55,5 +55,5 @@
                 xyz="-0.0547636346252869 0.0380939689802074 0.00933159404448308"
                 rpy="0 0 0"/>
-            <mass value="0.444820831236007"/>
+            <mass value="${0.444820831236007*lift_mass}"/>
             <inertia
                 ixx="0.000567192946271367"

File: stretch_control/urdf/stretch/stretch_right_wheel.xacro (robot description, xacro)
@@ -7,5 +7,5 @@
                 xyz="1.25554620866719E-07 3.54748938447003E-07 0.0239581106165018"
                 rpy="0 0 0" />
-            <mass value="0.00356714564938475" />
+            <mass value="${0.00356714564938475}" />
             <inertia ixx="0" ixy="0" ixz="0"
                      iyy="0" iyz="0"
@@ -40,16 +40,5 @@
         <axis xyz="0 0 1" />
     </joint>
-    <!-- Right Wheel Physical Properties for Gazebo -->
-    <gazebo reference="joint_right_wheel">
-        <mu1 value="200.0"/>
-        <mu2 value="100.0"/>
-        <kp value="10000000.0"/>
-        <kd value="1.0"/>
-        <material name="">
-            <color
-                rgba="0.792156862745098 0.819607843137255 0.933333333333333 1" />
-        </material>
-    </gazebo>
-    <!-- Gazebo transmission block for simulation -->
+    <!-- transmission block for ROS control -->
     <transmission name="trans_right_wheel">
         <type>transmission_interface/SimpleTransmission</type>
